Commit message: Pre-showcase

File: src/arm_description/robots/arm_description.urdf (robot description, URDF)
Before this commit: robot arm_description, 4 links, 3 joints
Links:
- added link ball, mass 0.028013; collision mesh filename=package://arm_description/meshes/ball.STL; visual mesh filename=package://arm_description/meshes/ball.STL
- link top: mass 0.25188 -> 0.22328
Joints:
- added joint ball_fixed: type fixed, parent top, child ball, origin xyz=0 0 0.1467 rpy=0 0 2.9027, axis 0 0 1
